File: NodeMCU ESP-32S Trinamic CNC.sch (KiCad schematic (older format))
At the start: 37 parts, among them J1 24V DC, J2 Micro_SD_Card, J3 X-AXIS, J4 Y-AXIS, J5 Z-AXIS, J6 SPINDLE OUT, J7 COOLANT RLY, J8 SPINDLE COOLANT RLY, K1 SRM-1C-SL-5VDC, K2 SRM-1C-SL-5VDC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

Commit message: First release with gerber files included.
Parts:
- removed J6: SPINDLE OUT, TerminalBlock:TerminalBlock_bornier-3_P5.08mm, symbol Connector:Screw_Terminal_01x03
- added D4, D5, D6, D7, D8: LED, LED_SMD:LED_0603_1608Metric, symbol Device:LED
- added J6: INPUTS/OUTPUTS, TerminalBlock:TerminalBlock_bornier-6_P5.08mm, symbol Connector:Screw_Terminal_01x06
- added R10: 1k, Resistor_SMD:R_0603_1608Metric, symbol Device:R
- added R11, R12, R13: 660R, Resistor_SMD:R_0603_1608Metric, symbol Device:R
- added R9: 4k7, Resistor_SMD:R_0603_1608Metric, symbol Device:R
- J2: symbol Connector:Micro_SD_Card -> NodeMCU-ESP-32S-Trinamic-CNC-rescue:Micro_SD_Card-Connector
Connections:
- net +24V: now also R9.1
- net +3V3: now also R11.1
- net +5V: now also R10.1
- net GND: now also D4.1 (K), D5.1 (K), D6.1 (K), D7.1 (K), D8.1 (K), J6.6 (Pin_6)
- net MIST: now also R12.1
- net PROBE: now also J6.1 (Pin_1)
- net SPINDLE_0_TO_10V: now also J6.5 (Pin_5)
- net SPINDLE_0_TO_5V: now also J6.4 (Pin_4)
- net SPINDLE_3v3_PWM: now also J6.3 (Pin_3)
- net SPINDLE_ENABLE: now also J6.2 (Pin_2), R13.1
- net at K1.11: now also J7.3 (Pin_3); no longer J7.2 (Pin_2)
- net at K1.14: now also J7.2 (Pin_2); no longer J7.3 (Pin_3)
- net at K2.11: now also J8.3 (Pin_3); no longer J8.2 (Pin_2)
- net at K2.14: now also J8.2 (Pin_2); no longer J8.3 (Pin_3)
- new net: D4.2 (A), R9.2
- new net: D5.2 (A), R10.2
- new net: D6.2 (A), R11.2
- new net: D7.2 (A), R12.2
- new net: D8.2 (A), R13.2
Other:
- note added: "POWER LED's"
